Commit message: new fixed links for calibration

File: cob_description/urdf/head_v3/head.urdf.xacro (robot description, xacro)
@@ -9,8 +9,34 @@
 	<include filename="$(find cob_description)/urdf/sensors/kinect.urdf.xacro" />
 	<xacro:macro name="cob_head_v3" params="name parent *origin">
-		<!-- joint between torso_upper_neck_tilt_link and head_axis_link -->
-		<joint name="${name}_axis_joint" type="revolute">
+		<!-- joint between torso_upper_neck_tilt_link and head_base_link -->
+		<joint name="head_base_joint" type="fixed">
 			<insert_block name="origin" />
 			<parent link="${parent}"/>
+			<child link="head_base_link"/>
+		</joint>
+		<link name="head_base_link">
+			<inertial>
+				<origin xyz="0 0 0" rpy="0 0 0"/>
+				<mass value="0.5"/>
+				<inertia ixx="0.01" ixy="0" ixz="0" iyy="0.01" iyz="0" izz="0.01" />
+			</inertial>
+			<visual>
+				<origin xyz="0 0 0" rpy="0 0 0" />
+				<geometry>
+					<mesh filename="package://cob_description/meshes/torso/head_cover.stl" />
+				</geometry>
+				<material name="IPA/Black" />
+			</visual>
+			<collision>
+				<origin xyz="0 0 0" rpy="0 0 0" />
+				<geometry>
+					<mesh filename="package://cob_description/meshes/torso/head_cover_collision.stl" />
+				</geometry>
+			</collision>
+		</link>
+		<!-- joint between head_base_link and head_axis_link -->
+		<joint name="${name}_axis_joint" type="revolute">
+			<parent link="head_base_link"/>
+			<origin xyz="0 0 0" rpy="0 0 0" />
 			<child link="${name}_axis_link"/>
 			<axis xyz="0 0 1" />
@@ -39,14 +65,40 @@
 			</collision>
 		</link>
+		<!-- joint between torso_upper_neck_tilt_link and head_base_link -->
+		<joint name="cam_reference_joint" type="fixed">
+			<origin xyz="${cam_ref_x} ${cam_ref_y} ${cam_ref_z}" rpy="${cam_ref_roll} ${cam_ref_pitch} ${cam_ref_yaw}" />
+			<parent link="head_axis_link"/>
+			<child link="cam_reference_link"/>
+		</joint>
+		<link name="cam_reference_link">
+			<inertial>
+				<origin xyz="0 0 0" rpy="0 0 0"/>
+				<mass value="0.5"/>
+				<inertia ixx="0.01" ixy="0" ixz="0" iyy="0.01" iyz="0" izz="0.01" />
+			</inertial>
+			<visual>
+				<origin xyz="0 0 0" rpy="0 0 0" />
+				<geometry>
+					<mesh filename="package://cob_description/meshes/torso/head_cover.stl" />
+				</geometry>
+				<material name="IPA/Black" />
+			</visual>
+			<collision>
+				<origin xyz="0 0 0" rpy="0 0 0" />
+				<geometry>
+					<mesh filename="package://cob_description/meshes/torso/head_cover_collision.stl" />
+				</geometry>
+			</collision>
+		</link>
 		<!-- left camera -->
-		<xacro:cob_prosilica_v0 name="${name}_color_camera_l" ros_topic="stereo/left" parent="${name}_axis_link">
-			<origin xyz="${cam_l_x} ${cam_l_y} ${cam_l_z}" rpy="${cam_l_roll} ${cam_l_pitch} ${cam_l_yaw}" />
+		<xacro:cob_prosilica_v0 name="${name}_color_camera_l" ros_topic="stereo/left" parent="cam_reference_link">
+			<origin xyz="0 0 0" rpy="0 0 0" />
 		</xacro:cob_prosilica_v0>
 		<!-- right camera -->
-		<xacro:cob_prosilica_v0 name="${name}_color_camera_r" ros_topic="stereo/right" parent="${name}_color_camera_l_link">
+		<xacro:cob_prosilica_v0 name="${name}_color_camera_r" ros_topic="stereo/right" parent="cam_reference_link">
 			<origin xyz="${cam_r_x} ${cam_r_y} ${cam_r_z}" rpy="${cam_r_roll} ${cam_r_pitch} ${cam_r_yaw}" />
 		</xacro:cob_prosilica_v0>
 		<!-- cam3d -->
-		<xacro:cob_kinect_v0 name="${name}_cam3d" ros_topic="cam3d" parent="${name}_color_camera_l_link">
+		<xacro:cob_kinect_v0 name="${name}_cam3d" ros_topic="cam3d" parent="cam_reference_link">
 			<origin xyz="${cam3d_x} ${cam3d_y} ${cam3d_z}" rpy="${cam3d_roll} ${cam3d_pitch} ${cam3d_yaw}" />
 		</xacro:cob_kinect_v0>

File: cob_description/urdf/torso_v1/torso.urdf.xacro (robot description, xacro)
@@ -7,11 +7,11 @@
 	<include filename="$(find cob_description)/urdf/torso_v1/torso.transmission.xacro" />
 	<xacro:macro name="cob_torso_v1" params="name parent *origin">
-		<!-- joint between base_link and arm_0_link -->
-		<joint name="${name}_0_joint" type="fixed" >
+		<!-- joint between base_link and torso_base_link -->
+		<joint name="${name}_base_joint" type="fixed" >
 			<insert_block name="origin" />
 			<parent link="${parent}" />
-			<child link="${name}_0_link" />
+			<child link="${name}_base_link" />
 		</joint>
-		<link name="${name}_0_link">
+		<link name="${name}_base_link">
 			<inertial>
 				<origin xyz="0 0 0" rpy="0 0 0"/>
@@ -20,5 +20,5 @@
 			</inertial>
 			<visual>
-				<origin xyz="0 0 -0.07" rpy="0 0 0" />
+				<origin xyz="0 0 -0.00" rpy="0 0 0" />
 				<geometry>
 					<cylinder radius="0" length="0"/>
@@ -36,5 +36,5 @@
 		<joint name="${name}_lower_neck_tilt_joint" type="revolute">
 			<origin xyz="0 0 0" rpy="0 0 0" />
-			<parent link="${name}_0_link"/>
+			<parent link="${name}_base_link"/>
 			<child link="${name}_lower_neck_tilt_link"/>
 			<axis xyz="0 0 1" />
@@ -123,18 +123,18 @@
 			</collision>
 		</link>
-		<!-- joint between torso_upper_neck_tilt_link and head_cover_link -->
-		<joint name="head_cover_joint" type="fixed">
-			<origin xyz="0 0 0" rpy="0 0 0" />
+		<!-- joint between torso_upper_neck_tilt_link and torso_upper_cover_link -->
+		<joint name="torso_upper_cover_joint" type="fixed">
+			<origin xyz="0 0 0" rpy="${M_PI} 0 0" />
 			<parent link="${name}_upper_neck_tilt_link"/>
-			<child link="head_cover_link"/>
+			<child link="torso_upper_cover_link"/>
 		</joint>
-		<link name="head_cover_link">
+		<link name="torso_upper_cover_link">
 			<inertial>
-				<origin xyz="0 0 0" rpy="${M_PI} 0 0"/>
+				<origin xyz="0 0 0" rpy="0 0 0"/>
 				<mass value="0.5"/>
 				<inertia ixx="0.01" ixy="0" ixz="0" iyy="0.01" iyz="0" izz="0.01" />
 			</inertial>
 			<visual>
-				<origin xyz="0 0 0" rpy="${M_PI} 0 0" />
+				<origin xyz="0 0 0" rpy="0 0 0" />
 				<geometry>
 					<mesh filename="package://cob_description/meshes/torso/head_cover.stl" />
@@ -143,5 +143,5 @@
 			</visual>
 			<collision>
-				<origin xyz="0 0 0" rpy="${M_PI} 0 0" />
+				<origin xyz="0 0 0" rpy="0 0 0" />
 				<geometry>
 					<mesh filename="package://cob_description/meshes/torso/head_cover_collision.stl" />

Commit message: fixed head model

File: cob_description/urdf/head_v3/head.urdf.xacro (robot description, xacro)
@@ -24,5 +24,5 @@
 				<origin xyz="0 0 0" rpy="0 0 0" />
 				<geometry>
-					<mesh filename="package://cob_description/meshes/torso/head_cover.stl" />
+					<box size="0.01 0.01 0.01"/>
 				</geometry>
 				<material name="IPA/Black" />
@@ -31,5 +31,5 @@
 				<origin xyz="0 0 0" rpy="0 0 0" />
 				<geometry>
-					<mesh filename="package://cob_description/meshes/torso/head_cover_collision.stl" />
+					<box size="0.01 0.01 0.01"/>
 				</geometry>
 			</collision>
@@ -80,5 +80,5 @@
 				<origin xyz="0 0 0" rpy="0 0 0" />
 				<geometry>
-					<mesh filename="package://cob_description/meshes/torso/head_cover.stl" />
+					<box size="0.01 0.01 0.01"/>
 				</geometry>
 				<material name="IPA/Black" />
@@ -87,5 +87,5 @@
 				<origin xyz="0 0 0" rpy="0 0 0" />
 				<geometry>
-					<mesh filename="package://cob_description/meshes/torso/head_cover_collision.stl" />
+					<box size="0.01 0.01 0.01"/>
 				</geometry>
 			</collision>
