Commit message: added cam_base_link

File: raw_description/urdf/torso/torso.urdf.xacro (robot description, xacro)
@@ -95,14 +95,43 @@
 			</collision>
 		</link>
+		<!-- joint between torso_upper_neck_tilt_link and head_axis_link -->
+		<joint name="cam_base_joint" type="fixed">
+			<origin xyz="0.0 0.0 0.0" rpy="0.0 0.0 0.0" />
+            <origin xyz="${cam_ref_x} ${cam_ref_y} ${cam_ref_z} "
+                rpy="${cam_ref_roll} ${cam_ref_pitch} ${cam_ref_yaw}" />
+   			<parent link="${name}_2_link"/>
+			<child link="cam_base_link"/>
+		</joint>
+		<link name="cam_base_link">
+			<inertial>
+				<origin xyz="0 0 0" rpy="0 0 0"/>
+				<mass value="0.1"/>
+				<inertia ixx="0.0001" ixy="0" ixz="0" iyy="0.0001" iyz="0" izz="0.0001" />
+			</inertial>
+			<visual>
+				<origin xyz="0 0 0" rpy="0 0 0" />
+				<geometry>
+					<box size="0.01 0.01 0.01"/>
+				</geometry>
+				<material name="IPA/LightGrey" />
+			</visual>
+			<collision>
+				<origin xyz="0 0 0" rpy="0 0 0" />
+				<geometry>
+					<box size="0.01 0.01 0.01"/>
+				</geometry>
+			</collision>
+		</link>
 		<!-- left camera -->
-		<xacro:cob_prosilica_v0 name="head_color_camera_l" ros_topic="stereo/left" parent="torso_2_link">
-			<origin xyz="${cam_l_x} ${cam_l_y} ${cam_l_z}" rpy="${cam_l_roll} ${cam_l_pitch} ${cam_l_yaw}" />
-		</xacro:cob_prosilica_v0>
+		<!--<xacro:cob_prosilica_v0 name="head_color_camera_l" ros_topic="stereo/left" parent="cam_base_link">-->
+			<!--<origin xyz="${cam_l_x} ${cam_l_y} ${cam_l_z}" rpy="${cam_l_roll} ${cam_l_pitch} ${cam_l_yaw}" />-->
+		<!--</xacro:cob_prosilica_v0>-->
 		<!-- right camera -->
-		<xacro:cob_prosilica_v0 name="head_color_camera_r" ros_topic="stereo/right" parent="torso_2_link">
-			<origin xyz="${cam_r_x} ${cam_r_y} ${cam_r_z}" rpy="${cam_r_roll} ${cam_r_pitch} ${cam_r_yaw}" />
-		</xacro:cob_prosilica_v0>
+		<!--<xacro:cob_prosilica_v0 name="head_color_camera_r" ros_topic="stereo/right" parent="cam_base_link">-->
+			<!--<origin xyz="${cam_r_x} ${cam_r_y} ${cam_r_z}" rpy="${cam_r_roll} ${cam_r_pitch} ${cam_r_yaw}" />-->
+		<!--</xacro:cob_prosilica_v0>-->
 		<!-- cam3d -->
-		<xacro:cob_kinect_v0 name="head_cam3d" ros_topic="cam3d" parent="torso_2_link">
+		<xacro:cob_kinect_v0 name="head_cam3d" ros_topic="cam3d"
+            parent="cam_base_link">
 			<origin xyz="${cam3d_x} ${cam3d_y} ${cam3d_z}" rpy="${cam3d_roll} ${cam3d_pitch} ${cam3d_yaw}" />
 		</xacro:cob_kinect_v0>
