Commit message: added fixed dummy link.  without it there is no transformation for calibration of torso

File: cob_description/urdf/torso_v1/torso.urdf.xacro (robot description, xacro)
@@ -7,8 +7,34 @@
 	<include filename="$(find cob_description)/urdf/torso_v1/torso.transmission.xacro" />
 	<xacro:macro name="cob_torso_v1" params="name parent *origin">
+		<!-- joint between base_link and arm_0_link -->
+		<joint name="${name}_0_joint" type="fixed" >
+			<insert_block name="origin" />
+			<parent link="${parent}" />
+			<child link="${name}_0_link" />
+		</joint>
+		<link name="${name}_0_link">
+			<inertial>
+				<origin xyz="0 0 0" rpy="0 0 0"/>
+				<mass value="0.01"/>
+				<inertia ixx="1" ixy="0" ixz="0" iyy="1" iyz="0" izz="1" />
+			</inertial>
+			<visual>
+				<origin xyz="0 0 -0.07" rpy="0 0 0" />
+				<geometry>
+					<cylinder radius="0" length="0"/>
+				</geometry>
+				<material name="Red" />
+			</visual>
+			<collision>
+				<origin xyz="0 0 0" rpy="0 0 0" />
+				<geometry>
+					<box size="0 0 0"/>
+				</geometry>
+			</collision>
+		</link>
 		<!-- joint between base_link and torso_lower_neck_tilt_link -->
 		<joint name="${name}_lower_neck_tilt_joint" type="revolute">
-			<insert_block name="origin" />
-			<parent link="${parent}"/>
+			<origin xyz="0 0 0" rpy="0 0 0" />
+			<parent link="${name}_0_link"/>
 			<child link="${name}_lower_neck_tilt_link"/>
 			<axis xyz="0 0 1" />

Commit message: unrotated head cover link as reference for head calibration

File: cob_description/urdf/torso_v1/torso.urdf.xacro (robot description, xacro)
@@ -125,5 +125,5 @@
 		<!-- joint between torso_upper_neck_tilt_link and head_cover_link -->
 		<joint name="head_cover_joint" type="fixed">
-			<origin xyz="0 0 0" rpy="${M_PI} 0 0" />
+			<origin xyz="0 0 0" rpy="0 0 0" />
 			<parent link="${name}_upper_neck_tilt_link"/>
 			<child link="head_cover_link"/>
@@ -131,10 +131,10 @@
 		<link name="head_cover_link">
 			<inertial>
-				<origin xyz="0 0 0" rpy="0 0 0"/>
+				<origin xyz="0 0 0" rpy="${M_PI} 0 0"/>
 				<mass value="0.5"/>
 				<inertia ixx="0.01" ixy="0" ixz="0" iyy="0.01" iyz="0" izz="0.01" />
 			</inertial>
 			<visual>
-				<origin xyz="0 0 0" rpy="0 0 0" />
+				<origin xyz="0 0 0" rpy="${M_PI} 0 0" />
 				<geometry>
 					<mesh filename="package://cob_description/meshes/torso/head_cover.stl" />
@@ -143,5 +143,5 @@
 			</visual>
 			<collision>
-				<origin xyz="0 0 0" rpy="0 0 0" />
+				<origin xyz="0 0 0" rpy="${M_PI} 0 0" />
 				<geometry>
 					<mesh filename="package://cob_description/meshes/torso/head_cover_collision.stl" />

Commit message: material red replaced

File: cob_description/urdf/torso_v1/torso.urdf.xacro (robot description, xacro)
@@ -24,5 +24,5 @@
 					<cylinder radius="0" length="0"/>
 				</geometry>
-				<material name="Red" />
+                <material name="IPA/DarkGrey" />
 			</visual>
 			<collision>
