Commit message: copy and paste error

File: raw_description/urdf/base_short/base.urdf.xacro (robot description, xacro)
@@ -102,5 +102,5 @@
     <!-- base laser rear -->
     <xacro:sick_s300_laser_v0 name="${name}_laser_rear" parent="${name}" ros_topic="laser_rear/scan_raw" update_rate="10" min_angle="-2.3562" max_angle="2.3562" >
-      <origin xyz="${laser_front_x} ${laser_front_y} ${laser_front_z}" rpy="${laser_front_roll} ${laser_front_pitch} ${laser_front_yaw}" />
+      <origin xyz="${laser_rear_x} ${laser_rear_y} ${laser_rear_z}" rpy="${laser_rear_roll} ${laser_rear_pitch} ${laser_rear_yaw}" />
     </xacro:sick_s300_laser_v0>
     <!-- cam3d -->
